File: hw/sch_pcb/BRIDGEADC01A.kicad_pcb (KiCad board)
At the start: 2 copper layers, 40.1 x 40.1 mm, 44 parts, among them J1 3÷5V, J10 POL, J11 ~RESET, J12 ~SYNC, J13 ~RDY, J14 ~CS, J15 SCLK, J16 DIN, J17 DOUT, J18 ~STANDBY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

Commit message: Edit production data
Other:
- net class Default removed
- net class Power removed
