File: hw/sch_pcb/BRIDGEADC01A.kicad_sch (KiCad schematic)
At the start: 44 parts, among them J1 3÷5V, J10 POL, J11 ~RESET, J12 ~SYNC, J13 ~RDY, J14 ~CS, J15 SCLK, J16 DIN, J17 DOUT, J18 ~STANDBY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

Commit message: Edit UST_ID
Parts:
- C1, C4, C5: UST_ID (none) -> 5c70984412875079b91f8865
- C2, C3, C6, C7: UST_ID (none) -> 5c70984712875079b91f8b4c
- D1, D2: UST_ID (none) -> 5c70984512875079b91f88ac
- L1, L2: UST_ID (none) -> 5c70984412875079b91f87fd
- R1, R2, R3: UST_ID (none) -> 5c70984612875079b91f899f
- U1: UST_ID (none) -> 5c70984612875079b91f8a06
- U2: UST_ID (none) -> 5c70984612875079b91f8a14
- Y1: UST_ID (none) -> 5c70984712875079b91f8b0d
Changed lines of the file:
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@@
   (symbol (lib_id "BRIDGEADC01A-rescue:GNDA") (at 227.33 78.74 0) (unit 1)
     (in_bom yes) (on_board yes)
-    (property "Reference" "#PWR?" (id 0) (at 227.33 85.09 0)
+    (property "Reference" "#PWR0101" (id 0) (at 227.33 85.09 0)
       (effects (font (size 1.27 1.27)) hide)
     )
@@
   (symbol (lib_id "BRIDGEADC01A-rescue:GNDA") (at 234.95 78.74 0) (unit 1)
     (in_bom yes) (on_board yes)
-    (property "Reference" "#PWR?" (id 0) (at 234.95 85.09 0)
+    (property "Reference" "#PWR0104" (id 0) (at 234.95 85.09 0)
       (effects (font (size 1.27 1.27)) hide)
     )
@@
   (symbol (lib_id "BRIDGEADC01A-rescue:GNDA") (at 257.81 78.74 0) (unit 1)
     (in_bom yes) (on_board yes)
-    (property "Reference" "#PWR?" (id 0) (at 257.81 85.09 0)
+    (property "Reference" "#PWR0103" (id 0) (at 257.81 85.09 0)
       (effects (font (size 1.27 1.27)) hide)
     )
@@
   (symbol (lib_id "BRIDGEADC01A-rescue:GNDA") (at 265.43 78.74 0) (unit 1)
     (in_bom yes) (on_board yes)
-    (property "Reference" "#PWR?" (id 0) (at 265.43 85.09 0)
+    (property "Reference" "#PWR0102" (id 0) (at 265.43 85.09 0)
       (effects (font (size 1.27 1.27)) hide)
     )
@@
       (effects (font (size 1.524 1.524)))
     )
+    (property "UST_ID" "5c70984512875079b91f88ac" (id 4) (at 252.73 30.48 0)
+      (effects (font (size 1.27 1.27)) hide)
+    )
     (pin "1")
     (pin "2")
@@
     (property "Datasheet" "" (id 3) (at 257.81 73.66 90)
       (effects (font (size 1.524 1.524)))
+    )
+    (property "UST_ID" "5c70984512875079b91f88ac" (id 4) (at 257.81 73.66 0)
+      (effects (font (size 1.27 1.27)) hide)
     )
     (pin "1")
@@
       (effects (font (size 1.524 1.524)))
     )
+    (property "UST_ID" "5c70984712875079b91f8b0d" (id 4) (at 171.45 86.36 0)
+      (effects (font (size 1.27 1.27)) hide)
+    )
     (pin "1")
     (pin "2")
@@
       (effects (font (size 1.524 1.524)))
     )
+    (property "UST_ID" "5c70984412875079b91f8865" (id 4) (at 227.33 73.66 0)
+      (effects (font (size 1.27 1.27)) hide)
+    )
     (pin "1")
     (pin "2")
@@
     (property "Datasheet" "" (id 3) (at 237.49 30.48 0)
       (effects (font (size 1.524 1.524)))
+    )
+    (property "UST_ID" "5c70984412875079b91f8865" (id 4) (at 237.49 30.48 0)
+      (effects (font (size 1.27 1.27)) hide)
     )
     (pin "1")
@@
       (effects (font (size 0.762 0.762)))
     )
+    (property "UST_ID" "5c70984612875079b91f899f" (id 4) (at 139.7 55.88 0)
+      (effects (font (size 1.27 1.27)) hide)
+    )
     (pin "1")
     (pin "2")
@@
       (effects (font (size 0.762 0.762)))
     )
+    (property "UST_ID" "5c70984612875079b91f899f" (id 4) (at 146.05 55.88 0)
+      (effects (font (size 1.27 1.27)) hide)
+    )
     (pin "1")
     (pin "2")
@@
       (effects (font (size 0.762 0.762)))
     )
+    (property "UST_ID" "5c70984612875079b91f899f" (id 4) (at 186.69 64.77 0)
+      (effects (font (size 1.27 1.27)) hide)
+    )
     (pin "1")
     (pin "2")
@@
       (effects (font (size 1.524 1.524)))
     )
+    (property "UST_ID" "5c70984712875079b91f8b4c" (id 4) (at 234.95 73.66 0)
+      (effects (font (size 1.27 1.27)) hide)
+    )
     (pin "1")
     (pin "2")
@@
     (property "Datasheet" "" (id 3) (at 245.11 30.48 0)
       (effects (font (size 1.524 1.524)))
+    )
+    (property "UST_ID" "5c70984712875079b91f8b4c" (id 4) (at 245.11 30.48 0)
+      (effects (font (size 1.27 1.27)) hide)
     )
     (pin "1")
@@
       (effects (font (size 1.524 1.524)))
     )
+    (property "UST_ID" "5c70984412875079b91f87fd" (id 4) (at 232.41 125.73 0)
+      (effects (font (size 1.27 1.27)) hide)
+    )
     (pin "1")
     (pin "2")
@@
       (effects (font (size 1.524 1.524)))
     )
+    (property "UST_ID" "5c70984412875079b91f87fd" (id 4) (at 245.11 69.85 0)
+      (effects (font (size 1.27 1.27)) hide)
+    )
     (pin "1")
     (pin "2")
@@
       (effects (font (size 1.524 1.524)))
     )
+    (property "UST_ID" "5c70984712875079b91f8b4c" (id 4) (at 59.69 107.95 0)
+      (effects (font (size 1.27 1.27)) hide)
+    )
     (pin "1")
     (pin "2")
@@
       (effects (font (size 1.524 1.524)))
     )
+    (property "UST_ID" "5c70984712875079b91f8b4c" (id 4) (at 87.63 46.99 0)
+      (effects (font (size 1.27 1.27)) hide)
+    )
     (pin "1")
     (pin "2")
@@
     (property "Datasheet" "" (id 3) (at 93.98 46.99 0)
       (effects (font (size 1.524 1.524)))
+    )
+    (property "UST_ID" "5c70984412875079b91f8865" (id 4) (at 93.98 46.99 0)
+      (effects (font (size 1.27 1.27)) hide)
     )
     (pin "1")
@@
       (effects (font (size 1.524 1.524)))
     )
+    (property "UST_ID" "5c70984612875079b91f8a06" (id 4) (at 72.39 58.42 0)
+      (effects (font (size 1.27 1.27)) hide)
+    )
     (pin "3")
     (pin "6")
@@
     (property "Datasheet" "" (id 3) (at 72.39 78.74 0)
       (effects (font (size 1.524 1.524)))
+    )
+    (property "UST_ID" "5c70984612875079b91f8a06" (id 4) (at 72.39 78.74 0)
+      (effects (font (size 1.27 1.27)) hide)
     )
     (pin "3")
@@
     )
     (property "Datasheet" "" (id 3) (at 132.08 88.9 0))
+    (property "UST_ID" "5c70984612875079b91f8a14" (id 4) (at 132.08 88.9 0)
+      (effects (font (size 1.27 1.27)) hide)
+    )
     (pin "1")
     (pin "10")
@@
     )
     (path "/00000000-0000-0000-0000-0000567a9d8e"
-      (reference "#PWR?") (unit 1) (value "GNDA") (footprint "")
+      (reference "#PWR0101") (unit 1) (value "GNDA") (footprint "")
+    )
+    (path "/00000000-0000-0000-0000-0000567aa489"
+      (reference "#PWR0102") (unit 1) (value "GNDA") (footprint "")
+    )
+    (path "/00000000-0000-0000-0000-0000567aa456"
+      (reference "#PWR0103") (unit 1) (value "GNDA") (footprint "")
     )
     (path "/00000000-0000-0000-0000-0000567aa423"
-      (reference "#PWR?") (unit 1) (value "GNDA") (footprint "")
-    )
-    (path "/00000000-0000-0000-0000-0000567aa456"
-      (reference "#PWR?") (unit 1) (value "GNDA") (footprint "")
-    )
-    (path "/00000000-0000-0000-0000-0000567aa489"
-      (reference "#PWR?") (unit 1) (value "GNDA") (footprint "")
+      (reference "#PWR0104") (unit 1) (value "GNDA") (footprint "")
     )
     (path "/00000000-0000-0000-0000-000055623093"
