File: hw/sch_pcb/BRIDGEADC01.kicad_sch (KiCad schematic)
At the start: 44 parts, among them J1 3÷5V, J10 POL, J11 ~RESET, J12 ~SYNC, J13 ~RDY, J14 ~CS, J15 SCLK, J16 DIN, J17 DOUT, J18 ~STANDBY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

Commit message: aktualizace repozitare
Other:
- title: NAME -> BRIDGEADC01
